File: devboard-stm32g030f6p6/devboard-stm32g030f6p6.kicad_pcb (KiCad board)
At the start: 2 copper layers, 17.8 x 26.7 mm, 22 parts, among them J1 USB_B_Micro, J2 Conn_ARM_JTAG_SWD_10, J3 Pins_Right, J4 Pins_Left, SW1 Reset, U1 STM32G030F6P6, U2 XC6206P332MR, Y1 32MHz

Commit message: More layout work
Parts:
- turned J2 to 90 degrees
Routing:
- net GND: track 0.00 -> 38.9 mm, vias 0 -> 14
- net Net-(FB1-Pad1): track 0.00 -> 12.0 mm
- net A0: track 0.00 -> 11.5 mm, vias 0 -> 1
- net +3V3: track 0.00 -> 9.41 mm
- net A7: track 0.00 -> 8.75 mm, vias 0 -> 1
- net A1: track 0.00 -> 8.68 mm, vias 0 -> 1
- net Net-(C2-Pad1): track 0.00 -> 6.25 mm
- net A6: track 0.00 -> 5.99 mm, vias 0 -> 1
- net A2: track 0.00 -> 5.87 mm, vias 0 -> 1
- net A5: track 0.00 -> 4.30 mm, vias 0 -> 1
- net Net-(C1-Pad1): track 0.00 -> 4.19 mm
- net A4: track 0.00 -> 3.99 mm, vias 0 -> 1
- net A3: track 0.00 -> 3.78 mm, vias 0 -> 1
- net +5V: track 0.00 -> 2.75 mm
- net Net-(J1-Pad6): track 0.00 -> 1.60 mm
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- added copper zone on In1.Cu, net GND
- added copper zone on In2.Cu, net GND
Other:
- copper layers 2 -> 4
- net class Default: clearance 0.2 -> 0.127; trace_width 0.25 -> 0.127; via_dia 0.8 -> 0.4; via_drill 0.4 -> 0.2
- rule trace_clearance: 0.2 -> 0.127
- rule trace_min: 0.2 -> 0.127
- rule via_min_drill: 0.3 -> 0.2

Commit message: Finish layout
Parts:
- added C7: 100n, Capacitor_SMD:C_0603_1608Metric, F.Cu at (115.4, 87.1)
- moved R4 3.58 mm to (114.4, 84.6)
- moved C5 2.95 mm to (115.6, 80.9), turned to 0 degrees
- moved C6 1.07 mm to (113.9, 82.7), turned to 90 degrees
- moved Y1 0.75 mm to (116.1, 83.6), turned to 90 degrees
- moved R2 0.64 mm to (117.0, 87.1)
- moved R1 0.13 mm to (113.9, 87.1)
- moved FB1 0.06 mm to (119.4, 77.5)
- moved FB2 0.06 mm to (119.4, 73.7)
Routing:
- net +3V3: track 9.41 -> 39.7 mm
- net NRESET: track 0.00 -> 22.0 mm, vias 0 -> 2
- net GND: track 38.9 -> 58.9 mm, vias 14 -> 31
- net SWDCLK: track 0.00 -> 15.5 mm, vias 0 -> 2
- net SWDIO: track 0.00 -> 14.7 mm, vias 0 -> 2
- net I2C_SCL: track 0.00 -> 12.9 mm
- net I2C_SDA: track 0.00 -> 12.4 mm
- net Net-(C5-Pad2): track 0.00 -> 10.3 mm
- net UART_RX: track 0.00 -> 9.12 mm, vias 0 -> 1
- net LED_USER: track 0.00 -> 8.35 mm, vias 0 -> 2
- net UART_TX: track 0.00 -> 7.35 mm
- net Net-(R4-Pad1): track 0.00 -> 4.17 mm
- net Net-(D2-Pad2): track 0.00 -> 2.82 mm
- net Net-(D1-Pad2): track 0.00 -> 2.61 mm
- net Net-(C6-Pad1): track 0.00 -> 2.20 mm
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Other:
- outline, holes or cut-outs redrawn
- board text added: "3.3V"
- board text added: "5V"
- board text added: "A0"
- board text added: "A1"
- board text added: "A2"
- board text added: "A3"
- board text added: "A4"
- board text added: "A5"
- board text added: "A6"
- board text added: "A7"
- board text added: "DevBoard"
- board text added: "Finomnis'"
- board text added: "GND"
- board text added: "GPIO"
- board text added: "I2C"
- board text added: "Power"
- board text added: "RX"
- board text added: "SCL"
- board text added: "SDA"
- board text added: "STM32G030F6"
- board text added: "TX"
- board text added: "UART"
