File: devboard-stm32g030f6p6/devboard-stm32g030f6p6.kicad_pcb (KiCad board)
At the start: 4 copper layers, 17.8 x 26.7 mm, 23 parts, among them J1 USB_B_Micro, J2 Conn_ARM_JTAG_SWD_10, J3 Pins_Right, J4 Pins_Left, SW1 Reset, U1 STM32G030F6P6, U2 XC6206P332MR, Y1 32MHz

Commit message: Fix oscillator being rotated by 90 degrees
Parts:
- moved C5 3.40 mm to (115.8, 84.3)
- moved R4 1.08 mm to (113.8, 83.7), turned to 90 degrees
- moved C6 0.83 mm to (113.8, 81.9)
- moved Y1 0.38 mm to (116.1, 83.2)
Connections:
- Y1 pad 1: GND -> Net-(C5-Pad2)
- Y1 pad 2: Net-(C5-Pad2) -> GND
- Y1 pad 3: GND -> Net-(C6-Pad1)
- Y1 pad 4: Net-(C6-Pad1) -> GND
Routing:
- net Net-(C5-Pad2): track 10.3 -> 7.19 mm

Commit message: Update 10p caps in pcb
Parts:
- C5, C6: value 12p -> 10p
Changed lines of the file:
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@@
       (effects (font (size 1 1) (thickness 0.15)))
     )
-    (fp_text value 12p (at 0 1.16 90) (layer F.Fab)
+    (fp_text value 10p (at 0 1.16 90) (layer F.Fab)
       (effects (font (size 1 1) (thickness 0.15)))
     )
@@
       (effects (font (size 1 1) (thickness 0.15)))
     )
-    (fp_text value 12p (at 0 1.16) (layer F.Fab)
+    (fp_text value 10p (at 0 1.16) (layer F.Fab)
       (effects (font (size 1 1) (thickness 0.15)))
     )

Commit message: Increase via size to 0.25mm
Parts:
- moved C6 0.45 mm to (113.9, 81.4)
Routing:
- net SWDCLK: track 15.5 -> 14.5 mm
- net A6: track 5.99 -> 6.72 mm
Other:
- net class Default: via_dia 0.4 -> 0.45; via_drill 0.2 -> 0.25

Commit message: Increase crystal bypass caps back up to 12p
Parts:
- C5, C6: value 10p -> 12p
Changed lines of the file:
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@@
       (effects (font (size 1 1) (thickness 0.15)))
     )
-    (fp_text value 10p (at 0 1.16 90) (layer F.Fab)
+    (fp_text value 12p (at 0 1.16 90) (layer F.Fab)
       (effects (font (size 1 1) (thickness 0.15)))
     )
@@
       (effects (font (size 1 1) (thickness 0.15)))
     )
-    (fp_text value 10p (at 0 1.16) (layer F.Fab)
+    (fp_text value 12p (at 0 1.16) (layer F.Fab)
       (effects (font (size 1 1) (thickness 0.15)))
     )
