File: devboard-stm32g030f6p6/devboard-stm32g030f6p6.sch (KiCad schematic (older format))
At the start: 23 parts, among them J1 USB_B_Micro, J2 Conn_ARM_JTAG_SWD_10, J3 Pins_Right, J4 Pins_Left, SW1 Reset, U1 STM32G030F6P6, U2 XC6206P332MR, Y1 32MHz

Commit message: Add board layout
Parts:
- removed C7: 100n, Capacitor_SMD:C_0603_1608Metric, symbol Device:C_Small
Connections:
- net A0: now also J3.1 (Pin_1); no longer J3.8 (Pin_8)
- net A1: now also J3.2 (Pin_2); no longer J3.7 (Pin_7)
- net A2: now also J3.3 (Pin_3); no longer J3.6 (Pin_6)
- net A3: now also J3.4 (Pin_4); no longer J3.5 (Pin_5)
- net A4: now also J3.5 (Pin_5); no longer J3.4 (Pin_4)
- net A5: now also J3.6 (Pin_6); no longer J3.3 (Pin_3)
- net A6: now also J3.7 (Pin_7); no longer J3.2 (Pin_2)
- net A7: now also J3.8 (Pin_8); no longer J3.1 (Pin_1)
- net I2C_SCL: now also J4.7 (Pin_7); no longer J4.5 (Pin_5)
- net I2C_SDA: now also J4.6 (Pin_6); no longer J4.4 (Pin_4)
- net UART_RX: now also J4.4 (Pin_4); no longer J4.7 (Pin_7)
- net UART_TX: now also J4.5 (Pin_5); no longer J4.6 (Pin_6)
Changed lines of the file:
@@
 Connection ~ 3150 1300
-$Comp
-L Device:C_Small C7
-U 1 1 618BDFE2
-P 4450 3050
-F 0 "C7" H 4358 3096 50  0000 R CNN
-F 1 "100n" H 4358 3005 50  0000 R CNN
-F 2 "Capacitor_SMD:C_0603_1608Metric" H 4450 3050 50  0001 C CNN
-F 3 "~" H 4450 3050 50  0001 C CNN
-	1    4450 3050
-	-1   0    0    -1
-$EndComp
-Connection ~ 4450 2950
-$Comp
-L power:GND #PWR0105
-U 1 1 618BEEB2
-P 4450 3150
-F 0 "#PWR0105" H 4450 2900 50  0001 C CNN
-F 1 "GND" H 4300 3050 50  0000 C CNN
-F 2 "" H 4450 3150 50  0001 C CNN
-F 3 "" H 4450 3150 50  0001 C CNN
-	1    4450 3150
-	1    0    0    -1
-$EndComp
 $Comp
 L Device:C_Small C4
@@
 	1    0    0    -1
 $EndComp
+Text GLabel 9650 2850 0    50   Input ~ 0
+A0
+Text GLabel 9650 2950 0    50   Input ~ 0
+A1
+Text GLabel 9650 3050 0    50   Input ~ 0
+A2
+Text GLabel 9650 3150 0    50   Input ~ 0
+A3
+Text GLabel 9650 3250 0    50   Input ~ 0
+A4
+Text GLabel 9650 3350 0    50   Input ~ 0
+A5
+Text GLabel 9650 3450 0    50   Input ~ 0
+A6
 Text GLabel 9650 3550 0    50   Input ~ 0
-A0
-Text GLabel 9650 3450 0    50   Input ~ 0
-A1
-Text GLabel 9650 3350 0    50   Input ~ 0
-A2
-Text GLabel 9650 3250 0    50   Input ~ 0
-A3
-Text GLabel 9650 3150 0    50   Input ~ 0
-A4
-Text GLabel 9650 3050 0    50   Input ~ 0
-A5
-Text GLabel 9650 2950 0    50   Input ~ 0
-A6
-Text GLabel 9650 2850 0    50   Input ~ 0
 A7
+Text GLabel 9650 4500 0    50   Input ~ 0
+I2C_SCL
+Text GLabel 9650 4400 0    50   Input ~ 0
+I2C_SDA
+Text GLabel 9650 4200 0    50   Input ~ 0
+UART_RX
 Text GLabel 9650 4300 0    50   Input ~ 0
-I2C_SCL
-Text GLabel 9650 4200 0    50   Input ~ 0
-I2C_SDA
-Text GLabel 9650 4500 0    50   Input ~ 0
-UART_RX
-Text GLabel 9650 4400 0    50   Input ~ 0
 UART_TX
 $Comp

Commit message: Finish layout
Parts:
- added C7: 100n, Capacitor_SMD:C_0603_1608Metric, symbol Device:C_Small
Connections:
- net +3V3: now also C7.1
- net GND: now also C7.2
Changed lines of the file:
@@
 Wire Wire Line
 	2250 800  2350 800
+$Comp
+L power:GND #PWR0105
+U 1 1 618BEEB2
+P 4450 3150
+F 0 "#PWR0105" H 4450 2900 50  0001 C CNN
+F 1 "GND" H 4300 3050 50  0000 C CNN
+F 2 "" H 4450 3150 50  0001 C CNN
+F 3 "" H 4450 3150 50  0001 C CNN
+	1    4450 3150
+	1    0    0    -1
+$EndComp
+Connection ~ 4450 2950
+$Comp
+L Device:C_Small C7
+U 1 1 618BDFE2
+P 4450 3050
+F 0 "C7" H 4358 3096 50  0000 R CNN
+F 1 "100n" H 4358 3005 50  0000 R CNN
+F 2 "Capacitor_SMD:C_0603_1608Metric" H 4450 3050 50  0001 C CNN
+F 3 "~" H 4450 3050 50  0001 C CNN
+	1    4450 3050
+	-1   0    0    -1
+$EndComp
 $EndSCHEMATC
